File: kicad/synthcart-ctrl.kicad_pcb (KiCad board)
At the start: 2 copper layers, 160 x 111.8 mm, 32 parts, among them J1 Joystick right, J2 Joystick right

Commit message: version 1.1.0 changes
- move resisitors for left DB9 port to the right of the port
- add 4mm mounting holes
- pixel art without dithering
Parts:
- removed the G*** at (156.5, 130.6)
- removed R1: 4.7K, Resistor_THT:R_Axial_DIN0207_L6.3mm_D2.5mm_P10.16mm_Horizontal
- added G***: LOGO, synthcart-ctrl:amp_no_dither, F.Cu at (155.4, 136.1)
- added REF**: MountingHole_4mm, MountingHole:MountingHole_4mm, F.Cu at (228.9, 148.8)
- added REF**: MountingHole_4mm, MountingHole:MountingHole_4mm, F.Cu at (228.9, 52.1)
- added REF**: MountingHole_4mm, MountingHole:MountingHole_4mm, F.Cu at (83.6, 148.8)
- added REF**: MountingHole_4mm, MountingHole:MountingHole_4mm, F.Cu at (83.6, 51.8)
- added Re: 4.7K, Resistor_THT:R_Axial_DIN0207_L6.3mm_D2.5mm_P10.16mm_Horizontal, F.Cu at (135.1, 48.3)
- J1, J2: value Joystick right -> DB9 female
- moved R2 46.2 mm to (140.2, 48.3)
- moved R3 3.05 mm to (172.2, 48.3)
- moved R4 3.05 mm to (177.3, 48.3)
- moved J1 0.51 mm to (107.4, 57.1)
- moved J2 0.51 mm to (193.8, 57.1)
Routing:
- net l_green: track 102.9 -> 118.5 mm
- net r_green: track 102.9 -> 115.9 mm
- net l_violet: track 25.7 -> 31.1 mm
- net r_white: track 103.9 -> 100.8 mm, vias 0 -> 1
- net r_violet: track 25.7 -> 28.3 mm
- net l_white: track 103.9 -> 102.9 mm, vias 0 -> 1
- net l_blue: track 86.8 -> 87.3 mm
- net r_blue: track 86.8 -> 87.3 mm
Other:
- board text added: "SYNTHCART CTRL v1.1.0 Controller for Synthcart by Sven Berthold Arweiler github.com/sarweiler/synthcart-ctrl"
- board text removed: "SYNTHCART CTRL v1.0.0 Controller for Synthcart by Sven Berthold Arweiler github.com/sarweiler/synthcart-ctrl"
